Commit message: Basic SLAM working

File: install/retail_assistant_bringup/share/retail_assistant_bringup/description/gazebo_control.xacro (robot description, xacro)
@@ -1,36 +1,21 @@
 <?xml version="1.0"?>
-<robot xmlns:xacro="http://ros.org/wiki/xacro" name="retail_assistant">
-  <!--
-    This plugin loads ros2_control inside Gazebo (gz sim).
-    It reads your controller configuration from the YAML file below.
-  -->
-  <gazebo>
-    <plugin name="gz_ros2_control" filename="libgz_ros2_control-system.so">
-      <parameters>$(find retail_assistant_bringup)/config/ros2_control.yaml</parameters>
-    </plugin>
-  </gazebo>
-  <!--
-    Define transmissions for each wheel joint so ros2_control
-    can command their velocities through Gazebo.
-  -->
-  <transmission name="left_wheel_transmission">
-    <type>transmission_interface/SimpleTransmission</type>
-    <joint name="left_wheel_rear_joint">
-      <hardwareInterface>hardware_interface/VelocityJointInterface</hardwareInterface>
-    </joint>
-    <actuator name="left_motor">
-      <hardwareInterface>hardware_interface/VelocityJointInterface</hardwareInterface>
-      <mechanicalReduction>1</mechanicalReduction>
-    </actuator>
-  </transmission>
-  <transmission name="right_wheel_transmission">
-    <type>transmission_interface/SimpleTransmission</type>
-    <joint name="right_wheel_rear_joint">
-      <hardwareInterface>hardware_interface/VelocityJointInterface</hardwareInterface>
-    </joint>
-    <actuator name="right_motor">
-      <hardwareInterface>hardware_interface/VelocityJointInterface</hardwareInterface>
-      <mechanicalReduction>1</mechanicalReduction>
-    </actuator>
-  </transmission>
+<robot xmlns:xacro="http://www.ros.org/wiki/xacro">
+    <gazebo>
+        <plugin name="diff_drive" filename="libgazebo_ros_diff_drive.so">
+            <!-- Wheel Information -->
+            <left_joint>left_wheel_rear_joint</left_joint>
+            <right_joint>right_wheel_rear_joint</right_joint>
+            <wheel_separation>0.5</wheel_separation>
+            <wheel_diameter>0.1</wheel_diameter>
+            <!-- Limits -->
+            <max_wheel_torque>200</max_wheel_torque>
+            <max_wheel_acceleration>10.0</max_wheel_acceleration>
+            <!-- Output -->
+            <odometry_frame>odom</odometry_frame>
+            <robot_base_frame>base_link</robot_base_frame>
+            <publish_odom>true</publish_odom>
+            <publish_odom_tf>true</publish_odom_tf>
+            <publish_wheel_tf>true</publish_wheel_tf>
+        </plugin>
+    </gazebo>
 </robot>

File: install/retail_assistant_bringup/share/retail_assistant_bringup/description/robot.urdf.xacro (robot description, xacro)
@@ -2,4 +2,5 @@
 <robot xmlns:xacro="http://ros.org/wiki/xacro" name="retail_assistant">
     <xacro:include filename= "robot_core.xacro"/>
-    <xacro:include filename="gazebo_control.xacro:"/>
+    <xacro:include filename="gazebo_control.xacro"/>
+    <xacro:include filename="lidar.xacro"/>
 </robot>

File: install/retail_assistant_bringup/share/retail_assistant_bringup/description/robot_core.xacro (robot description, xacro)
@@ -4,4 +4,7 @@
     <material name="white">
         <color rgba="1 1 1 1"/>
+    </material>
+     <material name="green">
+        <color rgba="0 1 0 1"/>
     </material>
     <material name="orange">
@@ -16,4 +19,11 @@
     <!--  Base LINk  -->
     <link name="base_link">
+    </link>
+    <joint name="base_footprint_joint" type="fixed">
+        <parent link="base_link"/>
+        <child link="base_footprint"/>
+        <origin xyz="0 0 0" rpy="0 0 0"/>
+    </joint>
+    <link name="base_footprint">
     </link>
     <joint name="chassis_joint" type="fixed">
@@ -32,5 +42,5 @@
         </visual>
          <collision>
-           <origin xyz="0.165 0 0.1524"/>
+            <origin xyz="0.165 0 0.2"/>
             <geometry>
                 <box size="0.3302 0.4572 0.3048"/>
@@ -41,4 +51,7 @@
         </xacro:inertial_box>
     </link>
+    <gazebo reference="chassis">
+      <material>Gazebo/Blue</material>
+    </gazebo>
     <!-- Left tread -->
 <!-- Left invisble wheel to  actually drive do not add collision-->
@@ -65,4 +78,7 @@
   </xacro:inertial_cylinder>
 </link>
+<gazebo reference="left_rear_wheel">
+   <material>Gazebo/Orange</material>
+</gazebo>
 <!-- Right tread -->
 <!-- Right invisble wheel to  actually drive do not add collision-->
@@ -89,11 +105,14 @@
   </xacro:inertial_cylinder>
 </link>
+<gazebo reference="right_rear_wheel">
+   <material>Gazebo/Orange</material>
+</gazebo>
 <!-- Right invisble wheel to  actually drive do not add collision-->
 <!-- caster wheel-->
-<joint name="caster_wheel_joint" type="continuous">
+<joint name="caster_wheel_joint" type="fixed">
   <parent link="chassis"/>
   <child link="caster_wheel"/>
   <origin xyz="0.25 0 0.05" />
-</joint>S
+</joint>
 <link name="caster_wheel">
   <visual>
@@ -112,3 +131,8 @@
   </xacro:inertial_sphere>
 </link>
+<gazebo reference="caster_wheel">
+   <material>Gazebo/Black</material>
+   <mu1 value="0.001"/>
+   <mu2 value="0.001"/>
+</gazebo>
 </robot>
