Commit message: change the robot model to look more like treads

File: install/retail_assistant_bringup/share/retail_assistant_bringup/description/gazebo_control_tracked.xacro (robot description, xacro)
@@ -2,8 +2,19 @@
 <robot xmlns:xacro="http://www.ros.org/wiki/xacro">
     <gazebo>
-        <plugin name="simple_tracked_vehicle" filename="libSimpleTrackedVehiclePlugin.so">
-            <body>chassis</body>
-            <left_track>left_track</left_track>
-            <right_track>right_track</right_track>
+        <plugin name="diff_drive" filename="libgazebo_ros_diff_drive.so">
+            <!-- Wheel Information -->
+            <left_joint>left_wheel_center_joint</left_joint>
+            <right_joint>right_wheel_center_joint</right_joint>
+            <wheel_separation>0.5</wheel_separation>
+            <wheel_diameter>0.13</wheel_diameter>
+            <!-- Limits -->
+            <max_wheel_torque>200</max_wheel_torque>
+            <max_wheel_acceleration>10.0</max_wheel_acceleration>
+            <!-- Output -->
+            <odometry_frame>odom</odometry_frame>
+            <robot_base_frame>base_link</robot_base_frame>
+            <publish_odom>true</publish_odom>
+            <publish_odom_tf>true</publish_odom_tf>
+            <publish_wheel_tf>true</publish_wheel_tf>
         </plugin>
     </gazebo>

File: install/retail_assistant_bringup/share/retail_assistant_bringup/description/robot.urdf.xacro (robot description, xacro)
@@ -3,5 +3,5 @@
     <xacro:include filename= "robot_core_treads.xacro"/>
     <xacro:include filename="gazebo_control_tracked.xacro"/>
-    <xacro:include filename="lidar.xacro"/>
+   <xacro:include filename="lidar.xacro"/>
     <xacro:include filename="imu.xacro"/>
 </robot>

File: install/retail_assistant_bringup/share/retail_assistant_bringup/description/robot_core_treads.xacro (robot description, xacro)
@@ -56,59 +56,163 @@
     <!-- Left tread -->
 <!-- Left invisble wheel to  actually drive do not add collision-->
-<link name="left_tread">
-  <visual>
-    <origin xyz="0.175 0.1051 0.0635"/><!-- placement of rectangle joint for tf-->
-    <geometry>
-      <box size="0.4572 0.05 0.127"/>
-    </geometry>
-    <material name="black"/>
+<joint name="left_wheel_center_joint" type="continuous">
+  <parent link="base_link"/>
+  <child link="left_center_wheel"/>
+  <origin xyz="0.065 0.25 0.05" rpy="-${pi/2} 0 0"/>
+  <axis xyz="0 0 1"/>
+</joint>
+<link name="left_center_wheel">
+  <visual>
+    <geometry>
+      <cylinder radius="0.065" length="0.04"/>
+    </geometry>
+    <material name="orange"/>
   </visual>
   <collision>
-    <origin xyz="0.175 0.1051 0.0635"/><!-- placement of rectangle joint for tf-->
-    <geometry>
-      <box size="0.4572 0.05 0.127"/>
-    </geometry>
-  </collision>
-  <xacro:inertial_box mass="1.0" x="0.4572" y="0.05" z="0.127">
-    <origin xyz="0 0.1651 0.0635"/>
-  </xacro:inertial_box>
-</link>
-<joint name="left_tread_joint" type="fixed">
-  <parent link="chassis"/>
-  <child link="left_tread"/>
-  <origin xyz="0 0.1651 0"/>
-  <axis xyz="0 1 0 "/>
-</joint>
-<gazebo reference="left_tread">
-   <material>Gazebo/Orange</material>
+    <geometry>
+      <cylinder radius="0.065" length="0.04"/>
+    </geometry>
+  </collision>
+  <xacro:inertial_cylinder mass="0.2" length="0.04" radius="0.065">
+    <origin xyz="0 0 0" rpy="0 0 0"/>
+  </xacro:inertial_cylinder>
+</link>
+<gazebo reference="left_center_wheel">
+   <material>Gazebo/Orange</material>
+</gazebo>
+<joint name="left_wheel_rear_joint" type="continuous">
+  <parent link="base_link"/>
+  <child link="left_rear_wheel"/>
+  <origin xyz="-0.065 0.25 0.05" rpy="-${pi/2} 0 0"/>
+  <axis xyz="0 0 1"/>
+</joint>
+<link name="left_rear_wheel">
+  <visual>
+    <geometry>
+      <cylinder radius="0.065" length="0.04"/>
+    </geometry>
+    <material name="orange"/>
+  </visual>
+  <collision>
+    <geometry>
+      <cylinder radius="0.065" length="0.04"/>
+    </geometry>
+  </collision>
+  <xacro:inertial_cylinder mass="0.2" length="0.04" radius="0.065">
+    <origin xyz="0 0 0" rpy="0 0 0"/>
+  </xacro:inertial_cylinder>
+</link>
+<gazebo reference="left_rear_wheel">
+   <material>Gazebo/Orange</material>
+   <mu1 value="0.001"/>
+   <mu2 value="0.001"/>
+</gazebo>
+<joint name="left_wheel_front_joint" type="continuous">
+  <parent link="base_link"/>
+  <child link="left_front_wheel"/>
+  <origin xyz="0.195 0.25 0.05" rpy="-${pi/2} 0 0"/>
+  <axis xyz="0 0 1"/>
+</joint>
+<link name="left_front_wheel">
+  <visual>
+    <geometry>
+      <cylinder radius="0.065" length="0.04"/>
+    </geometry>
+    <material name="orange"/>
+  </visual>
+  <collision>
+    <geometry>
+      <cylinder radius="0.065" length="0.04"/>
+    </geometry>
+  </collision>
+  <xacro:inertial_cylinder mass="0.2" length="0.04" radius="0.065">
+    <origin xyz="0 0 0" rpy="0 0 0"/>
+  </xacro:inertial_cylinder>
+</link>
+<gazebo reference="left_front_wheel">
+   <material>Gazebo/Orange</material>
+   <mu1 value="0.001"/>
+   <mu2 value="0.001"/>
 </gazebo>
 <!-- Right tread -->
 <!-- Right invisble wheel to  actually drive do not add collision-->
-<link name="right_tread">
-  <visual>
-    <origin xyz="0.175 -0.1051 0.0635"/>
-    <geometry>
-      <box size="0.4572 0.05 0.127"/>
-    </geometry>
-    <material name="black"/>
-  </visual>
-  <collision>
-    <origin xyz="0.175 -0.1051 0.0635"/>
-    <geometry>
-      <box size="0.4572 0.05 0.127"/>
-    </geometry>
-  </collision>
-  <xacro:inertial_box mass="1.0" x="0.4572" y="0.05" z="0.127">
-    <origin xyz="0 -0.1651 0.0635"/>
-  </xacro:inertial_box>
-</link>
-<joint name="right_tread_joint" type="fixed">
-  <parent link="chassis"/>
-  <child link="right_tread"/>
-  <origin xyz="0 -0.1651 0"/>
-  <axis xyz="0 1 0"/>
-</joint>
-<gazebo reference="right_tread">
-   <material>Gazebo/Orange</material>
+<joint name="right_wheel_center_joint" type="continuous">
+  <parent link="base_link"/>
+  <child link="right_center_wheel"/>
+  <origin xyz="0.065 -0.25 0.05" rpy="${pi/2} 0 0"/>
+  <axis xyz="0 0 -1"/>
+</joint>
+<link name="right_center_wheel">
+  <visual>
+    <geometry>
+      <cylinder radius="0.065" length="0.04"/>
+    </geometry>
+    <material name="orange"/>
+  </visual>
+    <collision>
+    <geometry>
+      <cylinder radius="0.065" length="0.04"/>
+    </geometry>
+  </collision>
+  <xacro:inertial_cylinder mass="0.2" length="0.04" radius="0.065">
+    <origin xyz="0 0 0" rpy=" 0 0 0"/>
+  </xacro:inertial_cylinder>
+</link>
+<gazebo reference="right_center_wheel">
+   <material>Gazebo/Orange</material>
+</gazebo>
+<joint name="right_wheel_front_joint" type="continuous">
+  <parent link="base_link"/>
+  <child link="right_front_wheel"/>
+  <origin xyz="0.195 -0.25 0.05" rpy="${pi/2} 0 0"/>
+  <axis xyz="0 0 -1"/>
+</joint>
+<link name="right_front_wheel">
+  <visual>
+    <geometry>
+      <cylinder radius="0.065" length="0.04"/>
+    </geometry>
+    <material name="orange"/>
+  </visual>
+    <collision>
+    <geometry>
+      <cylinder radius="0.065" length="0.04"/>
+    </geometry>
+  </collision>
+  <xacro:inertial_cylinder mass="0.2" length="0.04" radius="0.065">
+    <origin xyz="0 0 0" rpy=" 0 0 0"/>
+  </xacro:inertial_cylinder>
+</link>
+<gazebo reference="right_front_wheel">
+   <material>Gazebo/Orange</material>
+   <mu1 value="0.001"/>
+   <mu2 value="0.001"/>
+</gazebo>
+<joint name="right_wheel_rear_joint" type="continuous">
+  <parent link="base_link"/>
+  <child link="right_rear_wheel"/>
+  <origin xyz="-0.065 -0.25 0.05" rpy="${pi/2} 0 0"/>
+  <axis xyz="0 0 -1"/>
+</joint>
+<link name="right_rear_wheel">
+  <visual>
+    <geometry>
+      <cylinder radius="0.065" length="0.04"/>
+    </geometry>
+    <material name="orange"/>
+  </visual>
+    <collision>
+    <geometry>
+      <cylinder radius="0.065" length="0.04"/>
+    </geometry>
+  </collision>
+  <xacro:inertial_cylinder mass="0.2" length="0.04" radius="0.065">
+    <origin xyz="0 0 0" rpy=" 0 0 0"/>
+  </xacro:inertial_cylinder>
+</link>
+<gazebo reference="right_rear_wheel">
+   <material>Gazebo/Orange</material>
+   <mu1 value="0.001"/>
+   <mu2 value="0.001"/>
 </gazebo>
 <!-- Right invisble wheel to  actually drive do not add collision-->
