Commit message: working communication

File: install/retail_assistant_bringup/share/retail_assistant_bringup/description/fake_person_robot.xacro (robot description, xacro)
@@ -1,33 +1 @@
-<?xml version ="1.0"?>
-<robot xmlns:xacro="http://ros.org/wiki/xacro" name="moving_obstacle">
-  <link name="base_link">
-  </link>
-    <joint name="body" type="fixed">
-      <parent link="base_link" />
-      <child link="body_link" />
-      <origin xyz="0 0 0." rpy="0 0 0" />
-    </joint>
-    <link name="body_link">
-     <inertial>
-      <mass value="50" />
-      <origin xyz="0 0 0" />
-      <inertia ixx="10" iyy="10" izz="10" ixy="0" ixz="0" iyz="0" />
-    </inertial>
-    <visual>
-      <geometry><box size="0.4 0.4 1.0" /></geometry>
-      <material><color rgba="0.8 0 0 1" /></material>
-    </visual>
-    <collision>
-      <geometry><box size="0.4 0.4 1.0" /></geometry>
-    </collision>
-  </link>
-  <gazebo>
-    <plugin name="object_controller" filename="libgazebo_ros_planar_move.so">
-      <commandTopic>cmd_vel</commandTopic>
-      <odometryTopic>odom</odometryTopic>
-      <odometryFrame>fake_person_odom</odometryFrame>
-      <odometryRate>20.0</odometryRate>
-      <robotBaseFrame>base_link</robotBaseFrame>
-    </plugin>
-  </gazebo>
-</robot>
+/home/kendell/retail_assistant_ws/build/retail_assistant_bringup/description/fake_person_robot.xacro

File: install/retail_assistant_bringup/share/retail_assistant_bringup/description/gazebo_control.xacro (robot description, xacro)
@@ -1,18 +1 @@
-<?xml version="1.0"?>
-<robot xmlns:xacro="http://www.ros.org/wiki/xacro">
-    <gazebo>
-        <plugin name="diff_drive" filename="libgazebo_ros_diff_drive.so">
-            <left_joint>left_wheel_rear_joint</left_joint>
-            <right_joint>right_wheel_rear_joint</right_joint>
-            <wheel_separation>0.5</wheel_separation>
-            <wheel_diameter>0.1</wheel_diameter>
-            <max_wheel_torque>200</max_wheel_torque>
-            <max_wheel_acceleration>10.0</max_wheel_acceleration>
-            <odometry_frame>odom</odometry_frame>
-            <robot_base_frame>base_link</robot_base_frame>
-            <publish_odom>true</publish_odom><!--Make all these false to simulate doing slam with only the IMU-->
-            <publish_odom_tf>true</publish_odom_tf>
-            <publish_wheel_tf>true</publish_wheel_tf>
-        </plugin>
-    </gazebo>
-</robot>
+/home/kendell/retail_assistant_ws/build/retail_assistant_bringup/description/gazebo_control.xacro

File: install/retail_assistant_bringup/share/retail_assistant_bringup/description/gazebo_control_tracked.xacro (robot description, xacro)
@@ -1,21 +1 @@
-<?xml version="1.0"?>
-<robot xmlns:xacro="http://www.ros.org/wiki/xacro">
-    <gazebo>
-        <plugin name="diff_drive" filename="libgazebo_ros_diff_drive.so">
-            <!-- Wheel Information -->
-            <left_joint>left_wheel_center_joint</left_joint>
-            <right_joint>right_wheel_center_joint</right_joint>
-            <wheel_separation>0.5</wheel_separation>
-            <wheel_diameter>0.13</wheel_diameter>
-            <!-- Limits -->
-            <max_wheel_torque>200</max_wheel_torque>
-            <max_wheel_acceleration>10.0</max_wheel_acceleration>
-            <!-- Output -->
-            <odometry_frame>odom</odometry_frame>
-            <robot_base_frame>base_link</robot_base_frame>
-            <publish_odom>true</publish_odom>
-            <publish_odom_tf>true</publish_odom_tf>
-            <publish_wheel_tf>true</publish_wheel_tf>
-        </plugin>
-    </gazebo>
-</robot>
+/home/kendell/retail_assistant_ws/build/retail_assistant_bringup/description/gazebo_control_tracked.xacro

File: install/retail_assistant_bringup/share/retail_assistant_bringup/description/proximity.xacro (robot description, xacro)
@@ -1,142 +1 @@
-<?xml version="1.0"?>
-<robot xmlns:xacro="http://www.ros.org/wiki/xacro" name="retail_assistant">
-  <!-- parent chassis assumed to exist -->
-  <link name="ultrasonic_1_link">
-    <visual>
-            <geometry>
-                <box size="0.044 0.020 0.015"/>
-            </geometry>
-            <material name="green"/>
-    </visual>
-         <collision>
-            <origin xyz="0.165 0 0.2"/>
-            <geometry>
-                <box size="0.044 0.020 0.015"/>
-            </geometry>
-        </collision>
-        <xacro:inertial_box mass="0.010" x="0.3302" y="0.4572" z="0.3048">
-            <origin xyz="0 0 0" rpy="0 0 0"/>
-        </xacro:inertial_box>
-  </link>
-  <!-- Position the sensor link on the robot with a fixed joint -->
-  <joint name="ultrasonic_1_joint" type="fixed">
-    <parent link="chassis"/>
-    <child  link="ultrasonic_1_link"/>
-    <origin xyz="0.35 0 0.1" rpy="0 0 0"/>
-  </joint>
-  <!-- Gazebo extension: SDF sensor goes inside this block -->
-  <gazebo reference="ultrasonic_1_link">
-    <material>Gazebo/Green</material>
-    <sensor name="ultrasonic_1" type="ray">
-    <pose> 0 0 0 0 0 0</pose>
-      <always_on>true</always_on>
-      <visualize>true</visualize>
-      <update_rate>10</update_rate>
-      <ray>
-        <scan>
-          <horizontal>
-            <samples>13</samples>
-            <resolution>1</resolution>
-            <min_angle>-0.35</min_angle>
-            <max_angle>0.35</max_angle>
-          </horizontal>
-          <vertical>
-            <samples>7</samples>
-            <resolution>1</resolution>
-            <min_angle>-0.05</min_angle>
-            <max_angle>0.05</max_angle>
-          </vertical>
-        </scan>
-        <range>
-          <min>0.03</min>
-          <max>4.0</max>
-          <resolution>0.01</resolution>
-        </range>
-        <noise>
-          <type>gaussian</type>
-          <mean>0.0</mean>
-          <stddev>0.01</stddev>
-        </noise>
-      </ray>
-      <!-- Gazebo Classic plugin to publish ROS 2 Range -->
-      <plugin name="ultrasonic_sensor_1" filename="libgazebo_ros_ray_sensor.so">
-        <ros>
-          <!-- publishes on ultrasonic/front (since default is ~/out) -->
-          <argument>~/out:=/ultrasonic/front</argument>
-        </ros>
-        <output_type>sensor_msgs/Range</output_type>
-        <radiation_type>ultrasound</radiation_type>
-        <frame_name>ultrasonic_1_link</frame_name>
-      </plugin>
-    </sensor>
-  </gazebo>
-<link name="ultrasonic_2_link">
-    <visual>
-            <geometry>
-                <box size="0.044 0.020 0.015"/>
-            </geometry>
-            <material name="green"/>
-    </visual>
-         <collision>
-            <origin xyz="0.165 0 0.2"/>
-            <geometry>
-                <box size="0.044 0.020 0.015"/>
-            </geometry>
-        </collision>
-        <xacro:inertial_box mass="0.010" x="0.3302" y="0.4572" z="0.3048">
-            <origin xyz="0 0 0" rpy="0 0 0"/>
-        </xacro:inertial_box>
-  </link>
-  <!-- Position the sensor link on the robot with a fixed joint -->
-  <joint name="ultrasonic_2_joint" type="fixed">
-    <parent link="chassis"/>
-    <child  link="ultrasonic_2_link"/>
-    <origin xyz="-0.01 0 0.1" rpy="0 0 ${pi}"/>
-  </joint>
-  <!-- Gazebo extension: SDF sensor goes inside this block -->
-  <gazebo reference="ultrasonic_2_link">
-    <material>Gazebo/Green</material>
-    <sensor name="ultrasonic_2" type="ray">
-    <pose> 0 0 0 0 0 0</pose>
-      <always_on>true</always_on>
-      <visualize>true</visualize>
-      <update_rate>10</update_rate>
-      <ray>
-        <scan>
-          <horizontal>
-            <samples>13</samples>
-            <resolution>1</resolution>
-            <min_angle>-0.35</min_angle>
-            <max_angle>0.35</max_angle>
-          </horizontal>
-          <vertical>
-            <samples>7</samples>
-            <resolution>1</resolution>
-            <min_angle>-0.05</min_angle>
-            <max_angle>0.05</max_angle>
-          </vertical>
-        </scan>
-        <range>
-          <min>0.03</min>
-          <max>4.0</max>
-          <resolution>0.01</resolution>
-        </range>
-        <noise>
-          <type>gaussian</type>
-          <mean>0.0</mean>
-          <stddev>0.01</stddev>
-        </noise>
-      </ray>
-      <!-- Gazebo Classic plugin to publish ROS 2 Range -->
-      <plugin name="ultrasonic_sensor_2" filename="libgazebo_ros_ray_sensor.so">
-        <ros>
-          <!-- publishes on ultrasonic/front (since default is ~/out) -->
-          <argument>~/out:=/ultrasonic/back</argument>
-        </ros>
-        <output_type>sensor_msgs/Range</output_type>
-        <radiation_type>ultrasound</radiation_type>
-        <frame_name>ultrasonic_1_link</frame_name>
-      </plugin>
-    </sensor>
-  </gazebo>
-</robot>
+/home/kendell/retail_assistant_ws/build/retail_assistant_bringup/description/proximity.xacro

File: install/retail_assistant_bringup/share/retail_assistant_bringup/description/robot.urdf.xacro (robot description, xacro)
@@ -1,8 +1 @@
-<?xml version ="1.0"?>
-<robot xmlns:xacro="http://ros.org/wiki/xacro" name="retail_assistant">
-    <xacro:include filename= "robot_core_treads.xacro"/>
-    <xacro:include filename="gazebo_control_tracked.xacro"/>
-    <xacro:include filename="lidar.xacro"/>
-    <xacro:include filename="imu.xacro"/>
-    <xacro:include filename="proximity.xacro"/>
-</robot>
+/home/kendell/retail_assistant_ws/build/retail_assistant_bringup/description/robot.urdf.xacro

File: install/retail_assistant_bringup/share/retail_assistant_bringup/description/robot_core_treads.xacro (robot description, xacro)
@@ -1,220 +1 @@
-<?xml version ="1.0"?>
-<robot xmlns:xacro="http://ros.org/wiki/xacro">
-    <xacro:include filename="inertial_macros.xacro"/>
-    <material name="white">
-        <color rgba="1 1 1 1"/>
-    </material>
-     <material name="green">
-        <color rgba="0 1 0 1"/>
-    </material>
-    <material name="orange">
-        <color rgba="1 0.647 0 1"/>
-    </material>
-    <material name="blue">
-        <color rgba="0 0 1 1"/>
-    </material>
-    <material name="black">
-        <color rgba="0 0 0 1"/>
-    </material>
-    <!--  Base LINk  -->
-    <link name="base_link">
-    </link>
-    <joint name="base_footprint_joint" type="fixed">
-        <parent link="base_link"/>
-        <child link="base_footprint"/>
-        <origin xyz="0 0 0" rpy="0 0 0"/>
-    </joint>
-    <link name="base_footprint">
-    </link>
-    <joint name="chassis_joint" type="fixed">
-        <parent link="base_link"/>
-        <child link="chassis"/>
-        <origin xyz="-0.1 0 0"/>
-    </joint>
-<!--   Chassis    -->
-    <link name="chassis">
-        <visual>
-            <origin xyz="0.165 0 0.2"/>
-            <geometry>
-                <box size="0.3302 0.4572 0.3048"/>
-            </geometry>
-            <material name="blue"/>
-        </visual>
-         <collision>
-            <origin xyz="0.165 0 0.2"/>
-            <geometry>
-                <box size="0.3302 0.4572 0.3048"/>
-            </geometry>
-        </collision>
-        <xacro:inertial_box mass="4.5" x="0.3302" y="0.4572" z="0.3048">
-            <origin xyz="0.165 0 0.1524" rpy="0 0 0"/>
-        </xacro:inertial_box>
-    </link>
-    <gazebo reference="chassis">
-      <material>Gazebo/Blue</material>
-    </gazebo>
-    <!-- Left tread -->
-<!-- Left invisble wheel to  actually drive do not add collision-->
-<joint name="left_wheel_center_joint" type="continuous">
-  <parent link="base_link"/>
-  <child link="left_center_wheel"/>
-  <origin xyz="0.065 0.25 0.05" rpy="-${pi/2} 0 0"/>
-  <axis xyz="0 0 1"/>
-</joint>
-<link name="left_center_wheel">
-  <visual>
-    <geometry>
-      <cylinder radius="0.065" length="0.04"/>
-    </geometry>
-    <material name="orange"/>
-  </visual>
-  <collision>
-    <geometry>
-      <cylinder radius="0.065" length="0.04"/>
-    </geometry>
-  </collision>
-  <xacro:inertial_cylinder mass="0.2" length="0.04" radius="0.065">
-    <origin xyz="0 0 0" rpy="0 0 0"/>
-  </xacro:inertial_cylinder>
-</link>
-<gazebo reference="left_center_wheel">
-   <material>Gazebo/Orange</material>
-</gazebo>
-<joint name="left_wheel_rear_joint" type="continuous">
-  <parent link="base_link"/>
-  <child link="left_rear_wheel"/>
-  <origin xyz="-0.065 0.25 0.05" rpy="-${pi/2} 0 0"/>
-  <axis xyz="0 0 1"/>
-</joint>
-<link name="left_rear_wheel">
-  <visual>
-    <geometry>
-      <cylinder radius="0.065" length="0.04"/>
-    </geometry>
-    <material name="orange"/>
-  </visual>
-  <collision>
-    <geometry>
-      <cylinder radius="0.065" length="0.04"/>
-    </geometry>
-  </collision>
-  <xacro:inertial_cylinder mass="0.2" length="0.04" radius="0.065">
-    <origin xyz="0 0 0" rpy="0 0 0"/>
-  </xacro:inertial_cylinder>
-</link>
-<gazebo reference="left_rear_wheel">
-   <material>Gazebo/Orange</material>
-   <mu1 value="0.001"/>
-   <mu2 value="0.001"/>
-</gazebo>
-<joint name="left_wheel_front_joint" type="continuous">
-  <parent link="base_link"/>
-  <child link="left_front_wheel"/>
-  <origin xyz="0.195 0.25 0.05" rpy="-${pi/2} 0 0"/>
-  <axis xyz="0 0 1"/>
-</joint>
-<link name="left_front_wheel">
-  <visual>
-    <geometry>
-      <cylinder radius="0.065" length="0.04"/>
-    </geometry>
-    <material name="orange"/>
-  </visual>
-  <collision>
-    <geometry>
-      <cylinder radius="0.065" length="0.04"/>
-    </geometry>
-  </collision>
-  <xacro:inertial_cylinder mass="0.2" length="0.04" radius="0.065">
-    <origin xyz="0 0 0" rpy="0 0 0"/>
-  </xacro:inertial_cylinder>
-</link>
-<gazebo reference="left_front_wheel">
-   <material>Gazebo/Orange</material>
-   <mu1 value="0.001"/>
-   <mu2 value="0.001"/>
-</gazebo>
-<!-- Right tread -->
-<!-- Right invisble wheel to  actually drive do not add collision-->
-<joint name="right_wheel_center_joint" type="continuous">
-  <parent link="base_link"/>
-  <child link="right_center_wheel"/>
-  <origin xyz="0.065 -0.25 0.05" rpy="${pi/2} 0 0"/>
-  <axis xyz="0 0 -1"/>
-</joint>
-<link name="right_center_wheel">
-  <visual>
-    <geometry>
-      <cylinder radius="0.065" length="0.04"/>
-    </geometry>
-    <material name="orange"/>
-  </visual>
-    <collision>
-    <geometry>
-      <cylinder radius="0.065" length="0.04"/>
-    </geometry>
-  </collision>
-  <xacro:inertial_cylinder mass="0.2" length="0.04" radius="0.065">
-    <origin xyz="0 0 0" rpy=" 0 0 0"/>
-  </xacro:inertial_cylinder>
-</link>
-<gazebo reference="right_center_wheel">
-   <material>Gazebo/Orange</material>
-</gazebo>
-<joint name="right_wheel_front_joint" type="continuous">
-  <parent link="base_link"/>
-  <child link="right_front_wheel"/>
-  <origin xyz="0.195 -0.25 0.05" rpy="${pi/2} 0 0"/>
-  <axis xyz="0 0 -1"/>
-</joint>
-<link name="right_front_wheel">
-  <visual>
-    <geometry>
-      <cylinder radius="0.065" length="0.04"/>
-    </geometry>
-    <material name="orange"/>
-  </visual>
-    <collision>
-    <geometry>
-      <cylinder radius="0.065" length="0.04"/>
-    </geometry>
-  </collision>
-  <xacro:inertial_cylinder mass="0.2" length="0.04" radius="0.065">
-    <origin xyz="0 0 0" rpy=" 0 0 0"/>
-  </xacro:inertial_cylinder>
-</link>
-<gazebo reference="right_front_wheel">
-   <material>Gazebo/Orange</material>
-   <mu1 value="0.001"/>
-   <mu2 value="0.001"/>
-</gazebo>
-<joint name="right_wheel_rear_joint" type="continuous">
-  <parent link="base_link"/>
-  <child link="right_rear_wheel"/>
-  <origin xyz="-0.065 -0.25 0.05" rpy="${pi/2} 0 0"/>
-  <axis xyz="0 0 -1"/>
-</joint>
-<link name="right_rear_wheel">
-  <visual>
-    <geometry>
-      <cylinder radius="0.065" length="0.04"/>
-    </geometry>
-    <material name="orange"/>
-  </visual>
-    <collision>
-    <geometry>
-      <cylinder radius="0.065" length="0.04"/>
-    </geometry>
-  </collision>
-  <xacro:inertial_cylinder mass="0.2" length="0.04" radius="0.065">
-    <origin xyz="0 0 0" rpy=" 0 0 0"/>
-  </xacro:inertial_cylinder>
-</link>
-<gazebo reference="right_rear_wheel">
-   <material>Gazebo/Orange</material>
-   <mu1 value="0.001"/>
-   <mu2 value="0.001"/>
-</gazebo>
-<!-- Right invisble wheel to  actually drive do not add collision-->
-<!-- caster wheel-->
-</robot>
+/home/kendell/retail_assistant_ws/build/retail_assistant_bringup/description/robot_core_treads.xacro

File: src/retail_assistant_bringup/description/lidar.xacro (robot description, xacro)
@@ -3,8 +3,8 @@
   <joint name="lidar_joint" type="fixed">
     <parent link="chassis"/>
-    <child link="laser_frame"/>
+    <child link="laser"/>
     <origin xyz="0.2 0 0.3625" rpy="0 0 0"/>
 </joint>
-<link name="laser_frame">
+<link name="laser">
         <visual>
             <geometry>
@@ -22,33 +22,4 @@
         </xacro:inertial_cylinder>
     </link>
-    <gazebo reference="laser_frame">
-        <material>Gazebo/Green</material>
-        <sensor name="laser" type="ray">  <!--TODO Add comments explaning what all this means-->
-            <pose> 0 0 0 0 0 0</pose>
-            <visualize>true</visualize>
-            <update_rate>10</update_rate>
-            <ray>
-                <scan>
-                    <horizontal>
-                        <samples>360</samples>
-                        <resolution>1</resolution>
-                        <min_angle>-3.14</min_angle>
-                        <max_angle>3.14</max_angle>
-                    </horizontal>
-                </scan>
-                <range>
-                    <min>0.3</min>
-                    <max>12</max>
-                    <resolution>0.01</resolution>
-                </range>
-            </ray>
-            <plugin name="laser_controller" filename="libgazebo_ros_ray_sensor.so">
-                <ros>
-                    <argument>~/out:=scan</argument>
-                </ros>
-                <output_type>sensor_msgs/LaserScan</output_type>
-                <frame_name>laser_frame</frame_name>
-            </plugin>
-        </sensor>
-    </gazebo>
+<!--PLACE gazebo plugin for sim stuff if need-->
 </robot>
