Commit message: Most recent code on the pi working ultrasonics work in progress firebase upload

File: install/retail_assistant_bringup/share/retail_assistant_bringup/description/imu.xacro (robot description, xacro)
@@ -4,5 +4,5 @@
     <parent link="chassis"/>
     <child link="imu_frame"/>
-    <origin xyz="0.275 0 0.3625" rpy="0 0 0"/>
+    <origin xyz="0.275 0 0.279" rpy="0 0 0"/>
 </joint>
 <link name="imu_frame">

File: install/retail_assistant_bringup/share/retail_assistant_bringup/description/lidar.xacro (robot description, xacro)
@@ -4,5 +4,5 @@
     <parent link="chassis"/>
     <child link="laser"/>
-    <origin xyz="0.2 0 0.3625" rpy="0 0 0"/>
+    <origin xyz="0.05 0 0.3" rpy="0 0 0"/>
 </joint>
 <link name="laser">

File: install/retail_assistant_bringup/share/retail_assistant_bringup/description/proximity.xacro (robot description, xacro)
@@ -23,5 +23,5 @@
     <parent link="chassis"/>
     <child  link="ultrasonic_1_link"/>
-    <origin xyz="0.35 0 0.1" rpy="0 0 0"/>
+    <origin xyz="0.35 0 0.140" rpy="0 0 0"/>
   </joint>
   <!-- Gazebo extension: SDF sensor goes inside this block -->
@@ -92,5 +92,5 @@
     <parent link="chassis"/>
     <child  link="ultrasonic_2_link"/>
-    <origin xyz="-0.01 0 0.1" rpy="0 0 ${pi}"/>
+    <origin xyz="-0.015 0 0.140" rpy="0 0 ${pi}"/>
   </joint>
   <!-- Gazebo extension: SDF sensor goes inside this block -->

File: install/retail_assistant_bringup/share/retail_assistant_bringup/description/robot_core_treads.xacro (robot description, xacro)
@@ -37,5 +37,5 @@
             <origin xyz="0.165 0 0.2"/>
             <geometry>
-                <box size="0.3302 0.4572 0.3048"/>
+                <box size="0.381 0.3048 0.1524"/>
             </geometry>
             <material name="blue"/>
@@ -44,5 +44,5 @@
             <origin xyz="0.165 0 0.2"/>
             <geometry>
-                <box size="0.3302 0.4572 0.3048"/>
+                <box size="0.381 0.3048 0.1524"/>
             </geometry>
         </collision>
