Commit message: imu changes

File: src/retail_assistant_bringup/description/imu.xacro (robot description, xacro)
@@ -4,5 +4,5 @@
     <parent link="chassis"/>
     <child link="imu_frame"/>
-    <origin xyz="0.275 0 0.3625" rpy="0 0 0"/>
+    <origin xyz="0.275 0 0.3625" rpy="0 -0.624 0"/>
 </joint>
 <link name="imu_frame">
@@ -22,18 +22,3 @@
         </xacro:inertial_box>
     </link>
-    <gazebo reference="imu_frame"><!--Where to attach plugin in this case the link named imu_frame-->
-        <material>Gazebo/White</material>
-        <sensor name="imu_sensor" type="imu"><!--cretaes IMU sensor to simulate-->
-            <always_on>true</always_on><!--IMU is always on-->
-            <update_rate>30.0</update_rate><!-- How often IMU updates-->
-            <visualize>true</visualize><!--Whether to visualize in rviz-->
-            <plugin name="gazebo_ros_imu_sensor" filename="libgazebo_ros_imu_sensor.so"><!--Plugin connects gazebo and ros2-->
-                <ros>
-                    <namespace>/imu</namespace>
-                    <remapping>~/out:=data</remapping><!--Remaps output topic to /imu/data-->
-                </ros>
-                <gaussianNoise>0.0002</gaussianNoise>
-            </plugin><!--Adds noise to the IMU data to simulate real world-->
-        </sensor>
-    </gazebo>
 </robot>

Commit message: incorrect imu angle in urdf

File: src/retail_assistant_bringup/description/imu.xacro (robot description, xacro)
@@ -4,5 +4,5 @@
     <parent link="chassis"/>
     <child link="imu_frame"/>
-    <origin xyz="0.275 0 0.3625" rpy="0 -0.624 0"/>
+    <origin xyz="0.275 0 0.3625" rpy="0 0.624 0"/>
 </joint>
 <link name="imu_frame">

Commit message: resynchronizing with pi

File: src/retail_assistant_bringup/description/imu.xacro (robot description, xacro)
@@ -4,5 +4,5 @@
     <parent link="chassis"/>
     <child link="imu_frame"/>
-    <origin xyz="0.275 0 0.3625" rpy="0 0.624 0"/>
+    <origin xyz="0.275 0 0.3625" rpy="0 -0.624 0"/>
 </joint>
 <link name="imu_frame">

Commit message: changes made on the Pi

File: src/retail_assistant_bringup/description/imu.xacro (robot description, xacro)
@@ -4,5 +4,5 @@
     <parent link="chassis"/>
     <child link="imu_frame"/>
-    <origin xyz="0.275 0 0.3625" rpy="0 -0.624 0"/>
+    <origin xyz="0.275 0 0.3625" rpy="0 0 0"/>
 </joint>
 <link name="imu_frame">
